File: hardware/opencritter_pro/ESP-01.sch (KiCad schematic (older format))
At the start: 21 parts, among them J10 ESP Header, J11 ESP GPIO, SW5 GPIO0, SW6 RESET, U2 ESP8266EX, U3 CAT250, Y2 40Mhz

Commit message: DevKit1 Release
Added many new features and optimization for the new DevKit1
Parts:
- J10: value ESP Header -> ESP
Changed lines of the file:
@@
 P 1800 3000
 F 0 "J10" H 1800 3250 50  0000 C CNN
-F 1 "ESP Header" H 1800 2750 50  0000 C CNN
+F 1 "ESP" H 1800 2750 50  0000 C CNN
 F 2 "Pin_Headers:Pin_Header_Straight_2x04_Pitch2.54mm" H 1800 1800 50  0001 C CNN
 F 3 "" H 1800 1800 50  0001 C CNN
