File: hardware/oc_DevKit2/oc_DevKit2.kicad_pcb (KiCad board)
At the start: 2 copper layers, 35 x 43 mm, 40 parts, among them J3 I2C BUS, J4 USB_OTG, J5 IOPU SPI, J6 ESP, M1 Motor, SW1 GPIO0, SW2 RESET, SW3 Power, SW4 A, SW5 B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

Commit message: Inventory Update
Reworked stats, added new graphics, added inventory, updated energy system, reworked animation system.
Parts:
- moved C7 5.20 mm to (157.7, 55.8)
- moved D2 2.00 mm to (154.0, 54.5)
- moved R7 2.00 mm to (154.0, 57.4)
Routing:
- net +5V: track 29.0 -> 34.2 mm
- net +3V3: track 72.1 -> 67.6 mm
- net GND: track 83.7 -> 87.4 mm
Other:
- outline, holes or cut-outs redrawn
- board text added: "SuperMechaCow October 2017"
- board text removed: "Add secret circuit"
- board text removed: "Add signature"
- board text removed: "fix silk screen"
- board text removed: "move this cap so the three LEDS are evenly spaced"

Commit message: Lil Patch
Small changes. Updating for forthcoming Lite branch updates
Connections:
- R4 pad 1: +3V3 -> Net-(R4-Pad1)
- U1 pad 5: +3V3 -> Net-(R4-Pad1)
- U1 pad 7: +5V -> +3V3
- U1 pad 8: +5V -> (no net)
Routing:
- net Net-(R4-Pad1): track 0.00 -> 4.86 mm
- net +3V3: track 67.6 -> 63.5 mm
- net +5V: track 34.2 -> 32.8 mm, vias 2 -> 1
Changed lines of the file:
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@@
 (kicad_pcb (version 4) (host pcbnew 4.0.6)
   (general
-    (links 107)
+    (links 105)
     (no_connects 0)
-    (area 133.538095 48.766666 185.247619 96.100001)
+    (area 133.949999 52.949999 169.050001 96.050001)
     (thickness 1.6)
     (drawings 26)
-    (tracks 471)
+    (tracks 470)
     (zones 0)
     (modules 40)
-    (nets 26)
+    (nets 27)
   )
   (page A4)
@@
     (pad_to_mask_clearance 0)
     (aux_axis_origin 0 0)
-    (visible_elements 7FFFFF7F)
+    (visible_elements 7FFFEF7F)
     (pcbplotparams
       (layerselection 0x011fc_80000001)
@@
   (net 24 /ESP-01/RX)
   (net 25 /MOSI)
+  (net 26 "Net-(R4-Pad1)")
   (net_class Default "This is the default net class."
     (clearance 0.2)
@@
     (add_net "Net-(D2-Pad1)")
     (add_net "Net-(D3-Pad1)")
+    (add_net "Net-(R4-Pad1)")
     (add_net "Net-(R4-Pad2)")
     (add_net "Net-(R5-Pad1)")
@@
     (tags "capacitor 0805")
     (attr smd)
-    (fp_text reference C7 (at 1.9 1.5 450) (layer F.SilkS)
+    (fp_text reference C7 (at -1.3 -1.4 270) (layer F.SilkS)
       (effects (font (size 0.75 0.75) (thickness 0.15)))
     )
@@
     (tags "resistor 0805")
     (attr smd)
-    (fp_text reference D2 (at -3.1 0 270) (layer F.SilkS)
+    (fp_text reference D2 (at -1.7 -1.4 360) (layer F.SilkS)
       (effects (font (size 0.75 0.75) (thickness 0.15)))
     )
@@
     (tags "resistor 0805")
     (attr smd)
-    (fp_text reference D3 (at -3.1 0 270) (layer F.SilkS)
+    (fp_text reference D3 (at 0 -1.5 360) (layer F.SilkS)
       (effects (font (size 0.75 0.75) (thickness 0.15)))
     )
@@
     (fp_line (start 2.35 0.9) (end -2.35 0.9) (layer F.CrtYd) (width 0.05))
     (pad 1 smd rect (at -1.35 0 180) (size 1.5 1.3) (layers F.Cu F.Paste F.Mask)
-      (net 5 +3V3))
+      (net 26 "Net-(R4-Pad1)"))
     (pad 2 smd rect (at 1.35 0 180) (size 1.5 1.3) (layers F.Cu F.Paste F.Mask)
       (net 17 "Net-(R4-Pad2)"))
@@
     (tags "resistor 0805")
     (attr smd)
-    (fp_text reference R5 (at 3.3 0) (layer F.SilkS)
+    (fp_text reference R5 (at 0 1.5) (layer F.SilkS)
       (effects (font (size 0.75 0.75) (thickness 0.15)))
     )
@@
     (tags "resistor 0805")
     (attr smd)
-    (fp_text reference R7 (at -3.05 0 270) (layer F.SilkS)
+    (fp_text reference R7 (at 1.6 1.4 360) (layer F.SilkS)
       (effects (font (size 0.75 0.75) (thickness 0.15)))
     )
@@
     (tags "resistor 0805")
     (attr smd)
-    (fp_text reference R10 (at -3.1 0 270) (layer F.SilkS)
+    (fp_text reference R10 (at 0 -1.5 360) (layer F.SilkS)
       (effects (font (size 0.75 0.75) (thickness 0.15)))
     )
@@
       (net 12 /UART/D-))
     (pad 5 smd rect (at -1.95 0.75 180) (size 0.85 0.3) (layers F.Cu F.Paste F.Mask)
-      (net 5 +3V3))
+      (net 26 "Net-(R4-Pad1)"))
     (pad 6 smd rect (at -1.95 1.25 180) (size 0.85 0.3) (layers F.Cu F.Paste F.Mask)
       (net 5 +3V3))
     (pad 7 smd rect (at -1.25 1.95 270) (size 0.85 0.3) (layers F.Cu F.Paste F.Mask)
-      (net 4 +5V))
-    (pad 8 smd rect (at -0.75 1.95 270) (size 0.85 0.3) (layers F.Cu F.Paste F.Mask)
-      (net 4 +5V))
+      (net 5 +3V3))
+    (pad 8 smd rect (at -0.75 1.95 270) (size 0.85 0.3) (layers F.Cu F.Paste F.Mask))
     (pad 9 smd rect (at -0.25 1.95 270) (size 0.85 0.3) (layers F.Cu F.Paste F.Mask)
       (net 17 "Net-(R4-Pad2)"))
@@
     (tags "QFN 0.5")
     (attr smd)
-    (fp_text reference U4 (at 4 -2 90) (layer F.SilkS)
+    (fp_text reference U4 (at 3.2 0 180) (layer F.SilkS)
       (effects (font (size 1 1) (thickness 0.15)))
     )
@@
   (gr_line (start 161.6 55.2) (end 161.6 53.8) (layer F.SilkS) (width 0.1))
   (gr_line (start 161.6 53.8) (end 162.5 54.5) (layer F.SilkS) (width 0.1))
-  (gr_line (start 155.6 53.8) (end 156.5 54.5) (layer F.SilkS) (width 0.1))
-  (gr_line (start 155.6 55.2) (end 155.6 53.8) (layer F.SilkS) (width 0.1))
-  (gr_line (start 156.5 54.5) (end 155.6 55.2) (layer F.SilkS) (width 0.1))
+  (gr_line (start 153.6 53.8) (end 154.5 54.5) (layer F.SilkS) (width 0.1))
+  (gr_line (start 153.6 55.2) (end 153.6 53.8) (layer F.SilkS) (width 0.1))
+  (gr_line (start 154.5 54.5) (end 153.6 55.2) (layer F.SilkS) (width 0.1))
   (gr_line (start 147.5 54.5) (end 146.6 55.2) (layer F.SilkS) (width 0.1))
   (gr_line (start 146.6 53.8) (end 147.5 54.5) (layer F.SilkS) (width 0.1))
@@
   (gr_line (start 168 74) (end 168 96) (layer F.Fab) (width 0.2))
   (gr_line (start 135 74) (end 168 74) (layer F.Fab) (width 0.2))
+  (segment (start 146.8 68) (end 146.75 68.05) (width 0.1) (layer F.Cu) (net 0))
   (segment (start 141.12 63.55) (end 142.15 63.55) (width 0.25) (layer B.Cu) (net 1))
   (segment (start 140.744988 63.925012) (end 141.12 63.55) (width 0.25) (layer B.Cu) (net 1))
@@
   (segment (start 146.8 67.150002) (end 146.8 68.6016) (width 0.1) (layer B.Cu) (net 4))
   (segment (start 146.8 68.6016) (end 147.446197 69.247797) (width 0.1) (layer B.Cu) (net 4))
-  (segment (start 146.75 68.05) (end 147.25 68.05) (width 0.1) (layer F.Cu) (net 4))
-  (segment (start 146.8 67.150002) (end 146.8 68) (width 0.1) (layer F.Cu) (net 4))
-  (segment (start 146.8 68) (end 146.75 68.05) (width 0.1) (layer F.Cu) (net 4))
   (segment (start 144.85 63.55) (end 144.85 63.975) (width 0.1) (layer B.Cu) (net 4))
-  (via (at 146.8 67.150002) (size 0.6) (drill 0.4) (layers F.Cu B.Cu) (net 4))
   (segment (start 144.85 63.975) (end 146.8 65.925) (width 0.1) (layer B.Cu) (net 4))
   (segment (start 146.8 65.925) (end 146.8 67.150002) (width 0.1) (layer B.Cu) (net 4))
@@
   (segment (start 144.574996 62.699996) (end 144.85 62.975) (width 0.25) (layer B.Cu) (net 4))
   (segment (start 144.85 62.975) (end 144.85 63.55) (width 0.25) (layer B.Cu) (net 4))
+  (segment (start 147.425 68.75) (end 147.25 68.575) (width 0.1) (layer F.Cu) (net 5))
+  (segment (start 147.25 68.575) (end 147.25 68.05) (width 0.1) (layer F.Cu) (net 5))
   (segment (start 151.3 57.5) (end 151.300001 57.924265) (width 0.1) (layer B.Cu) (net 5))
   (segment (start 151.300001 57.924265) (end 151.300001 59.399999) (width 0.1) (layer B.Cu) (net 5))
@@
   (segment (start 135.5 62.69) (end 135.5 60.05) (width 0.1) (layer B.Cu) (net 5))
   (segment (start 135.5 60.05) (end 135.45 60) (width 0.1) (layer B.Cu) (net 5))
-  (segment (start 147.35 66) (end 148.2 66) (width 0.1) (layer F.Cu) (net 5))
-  (segment (start 148.2 66) (end 148.625001 66.425001) (width 0.1) (layer F.Cu) (net 5))
-  (segment (start 148.625001 66.425001) (end 148.625001 69.100001) (width 0.1) (layer F.Cu) (net 5))
-  (segment (start 148.625001 69.100001) (end 148.475 69.25) (width 0.1) (layer F.Cu) (net 5))
-  (segment (start 148.475 69.25) (end 147.95 69.25) (width 0.1) (layer F.Cu) (net 5))
   (segment (start 149.15 63.55) (end 150.03 63.55) (width 0.1) (layer B.Cu) (net 6))
   (segment (start 150.03 63.55) (end 150.180001 63.700001) (width 0.1) (layer B.Cu) (net 6))
@@
   (segment (start 136.939999 64.129999) (end 137.190001 64.380001) (width 0.1) (layer F.Cu) (net 25))
   (segment (start 137.190001 64.380001) (end 138.04 65.23) (width 0.1) (layer F.Cu) (net 25))
+  (segment (start 147.35 66) (end 148.2 66) (width 0.1) (layer F.Cu) (net 26))
+  (segment (start 148.2 66) (end 148.625001 66.425001) (width 0.1) (layer F.Cu) (net 26))
+  (segment (start 148.625001 66.425001) (end 148.625001 69.100001) (width 0.1) (layer F.Cu) (net 26))
+  (segment (start 148.625001 69.100001) (end 148.475 69.25) (width 0.1) (layer F.Cu) (net 26))
+  (segment (start 148.475 69.25) (end 147.95 69.25) (width 0.1) (layer F.Cu) (net 26))
   (zone (net 5) (net_name +3V3) (layer F.Cu) (hatch edge 0.508)
     (connect_pads (clearance 0.508))
