File: hardware/oc_DevKit2/oc_DevKit2.sch (KiCad schematic (older format))
At the start: 6 parts, among them J2 OLED, J3 I2C BUS, J4 USB_OTG, J5 IOPU SPI

Commit message: Lil Patch
Small changes. Updating for forthcoming Lite branch updates
Other:
- note added: "Add interupt to C button"
- note removed: "Add interupt to A button"
- note removed: "VERIFY HOW TO USE THE CP2102 AND IF THE SCHEMATIC IS RIGHT!\nESPECIALLY POWER!"
Changed lines of the file:
@@
 Text Label 5200 3200 0    60   ~ 0
 RESET
-Text Notes 1200 3250 0    60   ~ 0
-VERIFY HOW TO USE THE CP2102 AND IF THE SCHEMATIC IS RIGHT!\nESPECIALLY POWER!
 Text Notes 1200 4350 0    60   ~ 0
 Do the buttons need filter caps?
@@
 EndData
 $EndBitmap
-Text Notes 2050 2350 0    60   ~ 0
-Add interupt to A button
+Text Notes 950  1450 0    197  ~ 0
+Add interupt to C button
 $EndSCHEMATC
